File: SmartXeShieldForRaspberryPiZero2w/smartxeV6_small_board.kicad_pcb (KiCad board)
At the start: 2 copper layers, 48.8 x 19.1 mm, 15 parts

Commit message: updating the documentation
Connections:
- REF** pad 4: TCK_TO_TX_DUINO -> TMS_TO_RX_DUINO
- REF** pad 5: TMS_TO_RX_DUINO -> TCK_TO_TX_DUINO
- _ pad 10: TMS_TO_RX_DUINO -> TCK_TO_TX_DUINO
- _ pad 8: TCK_TO_TX_DUINO -> TMS_TO_RX_DUINO
Routing:
- net GND: track 6.47 -> 144.6 mm, vias 0 -> 2
- net VCC: track 50.0 -> 68.0 mm, vias 4 -> 5
- net SCK_PI: track 55.2 -> 46.6 mm
- net TCK_TO_TX_DUINO: track 19.9 -> 26.4 mm
- net TMS_TO_RX_DUINO: track 18.9 -> 15.9 mm
- net VCC_5V: track 64.1 -> 62.5 mm
- added copper zone on B.Cu, net GND
- added copper zone on F.Cu, net GND
Other:
- board size 48.8 x 19.1 mm -> 48.8 x 19.5 mm
- board text added: "If you use these two lines pi should go that way"
- board text added: "v1.1 {dblquote}ahhh that's why it doesn't work...{dblquote}"
- board text removed: "v0.33333333....*3~=1"
